File: _autosave-MCU_datalogger.kicad_sch (KiCad schematic)
At the start: 0 parts

Commit message: Added files
Other:
- title: (none) -> ${project_name}
Changed lines of the file:
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@@
 	(generator_version "9.0")
 	(paper "A4")
+	(title_block
+		(title "${project_name}")
+		(date "2025-11-17")
+	)
 	(sheet_instances
 		(path "/"
